Commit message: changed robot structure and made updates to inertia constants

File: my_robot/urdf/my_robot.xacro (robot description, xacro)
@@ -6,27 +6,27 @@
     	<origin xyz="0 0 0" rpy="0 0 0" />
         <parent link="robot_footprint" />
-        <child link="chassis" />
-    </joint>
-    <link name="chassis">
+        <child link="chassis_base" />
+    </joint>
+    <link name="chassis_base">
     	<pose>0 0 0.1 0 0 0</pose>
         <inertial>
-        	<mass value="15.0"/>
-            <origin xyz="0 0 0" rpy="0 0 0" />
-            <inertia
-            	ixx="0.1" ixy="0" ixz="0"
-                iyy="0.1" iyz="0"
-                izz="0.1"
-            />
-        </inertial>
-        <visual name="chassis_visual">
-        	<origin xyz="0 0 0" rpy="0 0 0" />
-        	<geometry>
-            	<box size="0.4 0.2 0.1" />
-            </geometry>
-        </visual>
-        <collision name="chassis_collision">
-        	<origin xyz="0 0 0" rpy="0 0 0" />
-        	<geometry>
-            	<box size="0.4 0.2 0.1" />
+        	<mass value="7.5"/>
+            <origin xyz="0 0 0" rpy="0 0 0"/>
+            <inertia
+            	ixx="0.1" ixy="0" ixz="0"
+                iyy="0.125" iyz="0"
+                izz="0.027"
+            />
+        </inertial>
+        <visual name="chassis_base_visual">
+        	<origin xyz="0 0 0" rpy="0 0 0"/>
+            <geometry>
+            	<box size="0.4 0.2 0.05" />
+            </geometry>
+        </visual>
+        <collision name="chassis_base_collision">
+        	<origin xyz="0 0 0" rpy="0 0 0" />
+        	<geometry>
+            	<box size="0.4 0.2 0.05" />
             </geometry>
         </collision>
@@ -102,5 +102,5 @@
     <joint name="left_wheel_hinge" type="continuous">
     	<origin xyz="0 0.15 0" rpy="0 0 0"/>
-        <parent link="chassis"/>
+        <parent link="chassis_base"/>
         <child link="left_wheel"/>
         <axis xyz="0 1 0" rpy="0 0 0"/>
@@ -110,5 +110,5 @@
     <joint name="right_wheel_hinge" type="continuous">
     	<origin xyz="0 -0.15 0" rpy="0 0 0"/>
-        <parent link="chassis"/>
+        <parent link="chassis_base"/>
         <child link="right_wheel"/>
         <axis xyz="0 1 0" rpy="0 0 0"/>
@@ -116,8 +116,93 @@
         <dynamics damping="1.0" friction="1.0"/>
 	</joint>
+    <link name="chassis_body">
+    	<pose>0 0 0.175 0 0 0</pose>
+        <inertial>
+        	<mass value="11.25"/>
+            <origin xyz="0 0 0" rpy="0 0 0" />
+            <inertia
+            	ixx="0.09" ixy="0" ixz="0"
+                iyy="0.122" iyz="0"
+                izz="0.1"
+            />
+        </inertial>
+        <visual name="chassis_body_visual">
+        	<origin xyz="0 0 0" rpy="0 0 0" />
+        	<geometry>
+            	<box size="0.3 0.2 0.1" />
+            </geometry>
+        </visual>
+        <collision name="chassis_body_collision">
+        	<origin xyz="0 0 0" rpy="0 0 0" />
+        	<geometry>
+            	<box size="0.3 0.2 0.1" />
+            </geometry>
+        </collision>
+	</link>
+    <joint name="chassis_body_base_joint" type="fixed">
+    	<origin xyz="0 0 0.075" rpy="0 0 0"/>
+        <parent link="chassis_base"/>
+        <child link="chassis_body"/>
+    </joint>
+    <link name="chassis_top">
+    	<pose>0 0 0.225 0 0 0</pose>
+        <inertial>
+        	<mass value="7.5"/>
+            <origin xyz="0 0 0" rpy="0 0 0"/>
+            <inertia
+            	ixx="0.1" ixy="0" ixz="0"
+                iyy="0.125" iyz="0"
+                izz="0.027"
+            />
+        </inertial>
+        <visual name="chassis_top_visual">
+        	<origin xyz="0 0 0" rpy="0 0 0"/>
+            <geometry>
+            	<box size="0.4 0.2 0.05" />
+            </geometry>
+        </visual>
+        <collision name="chassis_top_collision">
+        	<origin xyz="0 0 0" rpy="0 0 0" />
+        	<geometry>
+            	<box size="0.4 0.2 0.05" />
+            </geometry>
+        </collision>
+	</link>
+    <joint name="chassis_body_top_joint" type="fixed">
+    	<origin xyz="0 0 0.075" rpy="0 0 0"/>
+        <parent link="chassis_body"/>
+        <child link="chassis_top"/>
+    </joint>
     <link name="camera">
         <inertial>
-        	<mass value="0.1"/>
+        	<mass value="0.052"/>
             <box_inertia m="0.1" x="0.05" y="0.05" z="0.05" />
+            <inertia
+            	ixx="6.8e-7" ixy="0" ixz="0"
+                iyy="6.8e-7" iyz="0"
+                izz="6.8e-7"
+            />
+        </inertial>
+        <visual name="camera_visual">
+        	<origin xyz="0 0 0" rpy="0 0 0"/>
+            <geometry>
+                <sphere radius="0.025"/>
+            </geometry>
+        </visual>
+        <collision name="camera_collision">
+            <geometry>
+                <sphere radius="0.025"/>
+            </geometry>
+        </collision>
+    </link>
+    <joint type="fixed" name="camera_joint">
+    	<origin xyz="0.15 0 0" rpy="0 0 0"/>
+        <parent link="chassis_body"/>
+        <child link="camera"/>
+        <axis xyz="0 1 0"/>
+    </joint>
+    <link name="hokuyo">
+    	<inertial>
+        	<mass value="1e-5"/>
             <inertia
             	ixx="1e-6" ixy="0" ixz="0"
@@ -126,31 +211,4 @@
             />
         </inertial>
-        <visual name="camera_visual">
-        	<origin xyz="0 0 0" rpy="0 0 0"/>
-            <geometry>
-                <box size="0.05 0.05 0.05"/>
-            </geometry>
-        </visual>
-        <collision name="camera_collision">
-            <geometry>
-                <box size="0.05 0.05 0.05"/>
-            </geometry>
-        </collision>
-    </link>
-    <joint type="fixed" name="camera_joint">
-    	<origin xyz="0.2 0 0" rpy="0 0 0"/>
-        <parent link="chassis"/>
-        <child link="camera"/>
-        <axis xyz="0 1 0"/>
-    </joint>
-    <link name="hokuyo">
-    	<inertial>
-        	<mass value="1e-5"/>
-            <inertia
-            	ixx="1e-6" ixy="0" ixz="0"
-                iyy="1e-6" iyz="0"
-                izz="1e-6"
-            />
-        </inertial>
         <visual name="hokuyo_visual">
         	<origin xyz="0 0 0" rpy="0 0 0"/>
@@ -167,6 +225,6 @@
 	</link>
     <joint name="hokuyo_joint" type="fixed">
-    	<origin xyz="0.15 0 0.1" rpy="0 0 0"/>
-        <parent link="chassis"/>
+    	<origin xyz="0.15 0 0.075" rpy="0 0 0"/>
+        <parent link="chassis_top"/>
         <child link="hokuyo"/>
         <axis xyz="0 1 0"/>
@@ -178,9 +236,15 @@
         <material>Gazebo/Black</material>
     </gazebo>
-    <gazebo reference="chassis">
+    <gazebo reference="chassis_base">
+        <material>Gazebo/Black</material>
+    </gazebo>
+    <gazebo reference="chassis_body">
         <material>Gazebo/Red</material>
     </gazebo>
-    <gazebo reference="camera">
-        <material>Gazebo/SkyBlue</material>
+        <gazebo reference="chassis_top">
+        <material>Gazebo/Black</material>
+    </gazebo>
+	<gazebo reference="camera">
+        <material>Gazebo/Blue</material>
     </gazebo>
 </robot>

Commit message: added map.launch, RGBD camera and teleop package

File: my_robot/urdf/my_robot.xacro (robot description, xacro)
@@ -202,4 +202,11 @@
         <axis xyz="0 1 0"/>
     </joint>
+    <link name="camera_link_optical">
+    </link>
+    <joint name="camera_optical_joint" type="fixed">
+    	<origin xyz="0 0 0" rpy="-1.5707 0 -1.5707" />
+        <parent link="camera" />
+        <child link="camera_link_optical" />
+    </joint>
     <link name="hokuyo">
     	<inertial>
